File: V3/Schemetic/Trackerr_v3_Pcb/Trackerr_v3.kicad_sch (KiCad schematic)
At the start: 10 parts, among them P1 OLED 128X64 0.96, SW1 RST, U1 ABX00027, U2 ESP32_DevKit_V1_DOIT

Commit message: updated
Parts:
- removed P1: OLED 128X64 0.96, symbol SCHLIB_OLED-128X64-0.96_2025-02-08:OLED 128X64 0.96
- added +1: -, Connector_PinHeader_2.54mm:PinHeader_1x02_P2.54mm_Vertical, symbol Connector:Conn_01x02_Socket
- added J1, J2: Conn_01x01_Pin, Connector_PinHeader_2.54mm:PinHeader_1x01_P2.54mm_Vertical, symbol Connector:Conn_01x01_Pin
- added J3, J4: Conn_01x01_Socket, Connector_PinSocket_2.54mm:PinSocket_1x01_P2.54mm_Vertical, symbol Connector:Conn_01x01_Socket
- added J5, J6: Conn_01x02_Socket, Connector_PinSocket_2.54mm:PinSocket_1x02_P2.54mm_Vertical, symbol Connector:Conn_01x02_Socket
- added P1: OLED 128X64 0.96, PCBLIB_0.96-AND-1.3-I2C-OLED-SSD1306_2025-02-08:0.96 AND 1.3 I2C OLED SSD1306, symbol SCHLIB_OLED:OLED 128X64 0.96
- added U3: ~, PCBLIB_LM2596-DC-TO-DC-BUCK-CONVERTER-FOOTPRINT_2025-02-08:LM2596 DC TO DC BUCK CONVERTER FOOTPRINT, symbol LM2596 Step Down DC-DC Buck Converter:LM2596
- added U4: TP4056 Lithium Battery Charger Module, PCBLIB_BATTMODULE_2025-02-08:BATTMODULE, symbol SCHLIB_TP4056-Lithium-Battery-Charger-Module_2025-02-08:TP4056 Lithium Battery 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
- BZ1: footprint (none) -> Buzzer_Beeper:Buzzer_12x9.5RM7.6
- MODULE1, MODULE3: footprint (none) -> PCBLIB_LORA-SX1278-RA-02-WIRELESS-MODULE_2025-02-08:LORA SX1278 RA-02 WIRELESS MODULE
- MODULE2: footprint (none) -> PCBLIB_UBLOX-NEO-6M-GPS-MODULE_2025-02-08:UBLOX NEO 6M GPS MODULE
- Mode1, SW1, Select1: footprint (none) -> CUstom:SW_1825910-6-4
- U1: footprint ABX00027:MODULE_ABX00027 -> CUstom:MODULE_ABX00027
- U2: footprint ESP32_DevKit_V1_DOIT:esp32_devkit_v1_doit -> esp32_devkit_v1_doit:esp32_devkit_v1_doit
Connections:
- net GND: no longer BZ1.2 (-), Mode1.2, SW1.2, Select1.2
- net at MODULE3.3 (3V3), U2.16 (3V3): now also P1.2 (VDD)
- net at MODULE3.9 (GND), U2.17 (GND): now also BZ1.2 (-), MODULE3.1 (GND), MODULE3.16 (GND), MODULE3.2 (GND), Mode1.2, SW1.2, Select1.2, U2.14 (GND), J6.2 (Pin_2), P1.1 (GND)
- net at U2.29 (IO22): now also P1.3 (SCK)
- net at U2.26 (IO21): now also P1.4 (SDA)
- net at BZ1.1 (+): now also U2.8 (IO25); no longer U2.18 (IO15)
- net at MODULE1.1 (GND), MODULE1.16 (GND), MODULE1.2 (GND)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: now also MODULE1.9 (GND), J5.1 (Pin_1)
- net at MODULE2.2 (TX): now also U1.17 (RX); no longer U1.22 (D4)
- net at MODULE2.3 (RX): now also U1.16 (TX); no longer U1.21 (D3/PWM)
- net at U2.15 (VIN): now also J6.1 (Pin_1)
- net at U1.15 (VIN): now also J5.2 (Pin_2)
- new net: +1.1 (Pin_1), U4.6 (B+)
- new net: +1.2 (Pin_2), U4.5 (B-)
- new net: J1.1 (Pin_1), J3.1 (Pin_1), U3.4 (out+)
- new net: U3.1 (in-), U4.4 (Out-)
- new net: U3.2 (in+), U4.3 (OUt+)
- new net: J2.1 (Pin_1), J4.1 (Pin_1), U3.3 (out-)
Other:
- note added: "Supply"
